File: flightctrl.kicad_pcb (KiCad board)
At the start: 1 copper layers, 51 parts, among them J1 USB_OTG, SW1 SW_SPST, SW10 ROTARY_ENCODER_SWITCH, SW2 SW_SPST, SW3 SW_SPST, SW4 SW_SPST, SW5 SW_SPDT_MSM, SW6 ROTARY_ENCODER_SWITCH, SW7 ROTARY_ENCODER_SWITCH, SW8 ROTARY_ENCODER_SWITCH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

Commit message: update schematics
Parts:
- added C1: 10µ, Capacitors_ThroughHole:C_Radial_D5_L11_P2, B.Cu at (200.4, 96.5)
- added P1: CONN_02X03, Pin_Headers:Pin_Header_Straight_2x03_Pitch2.54mm, B.Cu at (198.1, 104.3)
Connections:
- J1 pad 4: Net-(J1-Pad4) -> (no net)
- SW7 pad 4: Net-(SW7-Pad4) -> (no net)
- SW7 pad 5: Net-(SW7-Pad5) -> (no net)
- SW8 pad 4: Net-(SW8-Pad4) -> (no net)
- SW8 pad 5: Net-(SW8-Pad5) -> (no net)
- SW9 pad 4: Net-(SW9-Pad4) -> (no net)
- SW9 pad 5: Net-(SW9-Pad5) -> (no net)
- U1 pad 19: Net-(U1-Pad19) -> (no net)
- U1 pad 22: Net-(U1-Pad22) -> (no net)
Routing:
- net Net-(P1-Pad5): track 0.00 -> 42.0 mm, vias 0 -> 2
- net +5V: track 315.1 -> 339.5 mm
- net GND: track 297.2 -> 318.6 mm
- net SW2_B: track 40.5 -> 53.7 mm, vias 0 -> 2
- net SW3_A: track 31.4 -> 41.6 mm, vias 0 -> 2
- net SW3_B: track 25.4 -> 33.6 mm, vias 0 -> 2
- net SW6: track 51.7 -> 53.7 mm
- net SW8: track 34.1 -> 36.1 mm
- net SW10b: track 103.8 -> 105.8 mm
- net SW7: track 68.7 -> 70.6 mm
- net SW10a: track 107.3 -> 109.2 mm
- net SW9: track 85.7 -> 87.6 mm
- net SW2_A: track 48.5 -> 47.5 mm
- net SW5_A: track 109.3 -> 110.1 mm
- net SW1_B: track 58.9 -> 58.2 mm
