File: flightctrl.sch (KiCad schematic (older format))
At the start: 53 parts, among them J1 USB_OTG, P1 CONN_02X03, SW1 SW_SPST, SW10 ROTARY_ENCODER_SWITCH, SW2 SW_SPST, SW3 SW_SPST, SW4 SW_SPST, SW5 SW_SPDT_MSM, SW6 ROTARY_ENCODER_SWITCH, SW7 ROTARY_ENCODER_SWITCH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

Commit message: update schematics
Parts:
- J1: symbol USB_OTG -> USB_OTG-RESCUE-flightctrl
- P1: footprint Pin_Headers:Pin_Header_Straight_2x03 -> Pin_Headers:Pin_Header_Straight_2x03_Pitch2.54mm
Changed lines of the file:
@@
 F 0 "P1" H 5400 2850 50  0000 C CNN
 F 1 "CONN_02X03" H 5400 2450 50  0000 C CNN
-F 2 "Pin_Headers:Pin_Header_Straight_2x03" H 5400 1450 50  0001 C CNN
+F 2 "Pin_Headers:Pin_Header_Straight_2x03_Pitch2.54mm" H 5400 1450 50  0001 C CNN
 F 3 "" H 5400 1450 50  0000 C CNN
 	1    5400 2650
@@
 	6400 1200 6700 1200
 $Comp
-L USB_OTG J1
+L USB_OTG-RESCUE-flightctrl J1
 U 1 1 5A2DEB92
 P 5950 6850
