File: input.sch (KiCad schematic (older format))
At the start: 24 parts, among them SW1 ROTARY_ENCODER_SWITCH, SW2 SW_SPST, SW3 SW_SPST, SW4 SW_SPST, SW5 ROTARY_ENCODER_SWITCH, SW6 SW_SPST, SW7 SW_SPST, SW8 SW_SPST

Commit message: update project for KiCAD 5.0, recreate/fix PCB
Parts:
- removed SW1, SW5: ROTARY_ENCODER_SWITCH, Button_Switch_THT:PEC11R-4xxxF-Sxxx, symbol Rotary_Encoder_Switch
- added SW7, SW8: Rotary_Encoder_Switch, Rotary_Encoder:RotaryEncoder_Alps_EC12E-Switch_Vertical_H20mm, symbol Device:Rotary_Encoder_Switch
- C6, C7, C8, C9: footprint Capacitors_SMD:C_0805 -> Capacitor_SMD:C_0805_2012Metric; symbol C -> flightctrl-rescue:C
- R10, R11, R12, R13, R14, R15, R16, R5, R6, R7, R8, R9: footprint Resistors_SMD:R_0805 -> Resistor_SMD:R_0805_2012Metric; symbol R -> flightctrl-rescue:R
- SW1: renamed from SW3; symbol SW_SPST -> flightctrl-rescue:SW_SPST
- SW2: renamed from SW6; symbol SW_SPST -> flightctrl-rescue:SW_SPST
- SW3: renamed from SW2; symbol SW_SPST -> flightctrl-rescue:SW_SPST
- SW4: renamed from SW7; symbol SW_SPST -> flightctrl-rescue:SW_SPST
- SW5: renamed from SW4; symbol SW_SPST -> flightctrl-rescue:SW_SPST
- SW6: renamed from SW8; symbol SW_SPST -> flightctrl-rescue:SW_SPST
Connections:
- net +5V: now also SW7.4, SW8.4
- net GND: now also SW7.2 (C), SW8.2 (C)
- net SW7_A: now also SW7.1 (A)
- net SW7_B: now also SW7.3 (B)
- net SW7_C: now also SW7.5
- net SW8_A: now also SW8.1 (A)
- net SW8_B: now also SW8.3 (B)
- net SW8_C: now also SW8.5
