File: output.sch (KiCad schematic (older format))
At the start: 24 parts, among them J2 CONN_01X02, J3 CONN_01X02, J4 CONN_01X02, J5 CONN_01X02, J6 CONN_01X02, J7 CONN_01X02, Q1 2N7000, Q2 2N7000, Q3 2N7000, Q4 2N7000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

Commit message: update project for KiCAD 5.0, recreate/fix PCB
Parts:
- J2, J3, J4, J5, J6, J7: footprint Terminal_Blocks:TerminalBlock_bornier-2_P5.08mm -> TerminalBlock:TerminalBlock_bornier-2_P5.08mm; symbol CONN_01X02 -> flightctrl-rescue:CONN_01X02
- Q1, Q2, Q3, Q4, Q5, Q7: footprint TO_SOT_Packages_THT:TO-92_Rugged -> Package_TO_SOT_THT:TO-92_HandSolder; symbol Q_NMOS_SGD -> flightctrl-rescue:Q_NMOS_SGD
- R17, R18, R19, R20, R21, R22, R23, R24, R25, R27, R29, R30: footprint Resistors_SMD:R_0805 -> Resistor_SMD:R_0805_2012Metric; symbol R -> flightctrl-rescue:R
